File: _autosave-SIM808_CIRCUIT.kicad_pcb (KiCad board)
At the start: 2 copper layers, 94 x 49.7 mm, 29 parts, among them J1 USB_B_Micro, J2 SMA-J-P-H-ST-EM1, J3 SIM_Card, J4 AVR-ISP-6, SW1 SW_Push, SW2 SW_Push, U1 MCP73811T-420I-OT, U2 SIM808, U3 74ABT125D, U4 ATmega328-AU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

Commit message: routed VRTC and RING line
Routing:
- net PWRKEY: track 0.00 -> 82.8 mm, vias 0 -> 2
- net VRTC: track 0.00 -> 18.5 mm, vias 0 -> 2
Changed lines of the file:
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@@
     (thickness 1.6)
     (drawings 7)
-    (tracks 575)
+    (tracks 602)
     (zones 0)
     (modules 29)
@@
   (gr_line (start 50.8 58.42) (end 144.78 58.42) (layer Edge.Cuts) (width 0.05))
   (gr_line (start 50.8 105.156) (end 50.8 58.42) (layer Edge.Cuts) (width 0.05))
+  (segment (start 77.408 81.152) (end 75.056 81.152) (width 0.25) (layer F.Cu) (net 1))
+  (segment (start 75.056 81.152) (end 74.422 80.518) (width 0.25) (layer F.Cu) (net 1))
+  (via (at 74.422 80.518) (size 0.8) (drill 0.4) (layers F.Cu B.Cu) (net 1))
+  (segment (start 74.422 81.083685) (end 74.803 81.464685) (width 0.25) (layer B.Cu) (net 1))
+  (segment (start 74.422 80.518) (end 74.422 81.083685) (width 0.25) (layer B.Cu) (net 1))
+  (segment (start 74.803 81.464685) (end 74.803 85.598) (width 0.25) (layer B.Cu) (net 1))
+  (segment (start 74.803 85.598) (end 79.121 89.916) (width 0.25) (layer B.Cu) (net 1))
+  (segment (start 79.121 89.916) (end 83.058 89.916) (width 0.25) (layer B.Cu) (net 1))
+  (via (at 83.058 89.916) (size 0.8) (drill 0.4) (layers F.Cu B.Cu) (net 1))
   (segment (start 140.612 77.017) (end 134.112 77.017) (width 0.25) (layer F.Cu) (net 2))
   (segment (start 111.506263 86.662237) (end 111.506263 88.391737) (width 0.25) (layer F.Cu) (net 2))
@@
   (segment (start 71.7065 93.2665) (end 71.7065 94.742) (width 0.25) (layer F.Cu) (net 25))
   (segment (start 71.755 93.218) (end 71.7065 93.2665) (width 0.25) (layer F.Cu) (net 25))
+  (segment (start 77.408 72.152) (end 89.424 72.152) (width 0.25) (layer F.Cu) (net 26))
+  (segment (start 89.424 72.152) (end 96.266 78.994) (width 0.25) (layer F.Cu) (net 26))
+  (segment (start 96.266 78.994) (end 96.266 80.01) (width 0.25) (layer F.Cu) (net 26))
+  (via (at 96.393 80.01) (size 0.8) (drill 0.4) (layers F.Cu B.Cu) (net 26))
+  (segment (start 96.266 80.01) (end 96.393 80.01) (width 0.25) (layer F.Cu) (net 26))
+  (segment (start 96.958685 80.01) (end 100.838 83.889315) (width 0.25) (layer B.Cu) (net 26))
+  (segment (start 96.393 80.01) (end 96.958685 80.01) (width 0.25) (layer B.Cu) (net 26))
+  (segment (start 100.838 83.889315) (end 100.838 89.281) (width 0.25) (layer B.Cu) (net 26))
+  (segment (start 100.838 89.281) (end 104.648 93.091) (width 0.25) (layer B.Cu) (net 26))
+  (segment (start 104.648 93.091) (end 114.935 93.091) (width 0.25) (layer B.Cu) (net 26))
+  (via (at 114.935 93.091) (size 0.8) (drill 0.4) (layers F.Cu B.Cu) (net 26))
+  (segment (start 114.935 93.091) (end 117.856 93.091) (width 0.25) (layer F.Cu) (net 26))
+  (segment (start 117.856 93.091) (end 118.999 94.234) (width 0.25) (layer F.Cu) (net 26))
+  (segment (start 118.999 94.234) (end 125.73 94.234) (width 0.25) (layer F.Cu) (net 26))
+  (segment (start 125.73 94.234) (end 131.318 88.646) (width 0.25) (layer F.Cu) (net 26))
+  (segment (start 131.318 85.471) (end 134.112 82.677) (width 0.25) (layer F.Cu) (net 26))
+  (segment (start 131.318 88.646) (end 131.318 85.471) (width 0.25) (layer F.Cu) (net 26))
+  (segment (start 134.112 82.677) (end 140.612 82.677) (width 0.25) (layer F.Cu) (net 26))
   (segment (start 132.697787 72.517) (end 134.112 72.517) (width 0.25) (layer F.Cu) (net 27))
   (segment (start 123.933 71.696) (end 123.933 69.615) (width 0.25) (layer F.Cu) (net 27))
