File: _autosave-SIM808_CIRCUIT.kicad_pcb (KiCad board)
At the start: 2 copper layers, 94 x 49.7 mm, 34 parts, among them J1 USB_B_Micro, J2 SMA-J-P-H-RA-TH1, J3 693012040811, J4 AVR-ISP-6, J5 U.FL-R-SMT(01), SW1 SW_Push, SW2 SW_Push, U1 MCP73811T-420I-OT, U2 SIM808, U3 74ABT125D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

Commit message: v1 sample
Parts:
- added REF**: OSHW-Logo2_14.6x12mm_SilkScreen, Symbol:OSHW-Logo2_14.6x12mm_SilkScreen, B.Cu at (98.9, 90.2)
- added REF**: OSHW-Logo2_14.6x12mm_SilkScreen, Symbol:OSHW-Logo2_14.6x12mm_SilkScreen, F.Cu at (66.7, 84.1)
Routing:
- net GND: track 289.9 -> 300.1 mm, vias 1 -> 3
Other:
- board text added: "BY: JACK MCLEANS"
- board text added: "TRACK BOARD"
