File: SIM808_CIRCUIT.kicad_pcb (KiCad board)
At the start: 2 copper layers, 94 x 49.7 mm, 29 parts, among them J1 USB_B_Micro, J2 SMA-J-P-H-ST-EM1, J3 SIM_Card, J4 AVR-ISP-6, SW1 SW_Push, SW2 SW_Push, U1 MCP73811T-420I-OT, U2 SIM808, U3 74ABT125D, U4 ATmega328-AU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

Commit message: Final routing attempt
Routing:
- net PWRKEY: track 0.00 -> 82.8 mm, vias 0 -> 2
- net SIM_RXD: track 0.00 -> 80.2 mm, vias 0 -> 2
- net Net-(J2-Pad1): track 0.00 -> 77.2 mm, vias 0 -> 2
- net SIM_RST: track 0.00 -> 43.0 mm, vias 0 -> 4
- net RING: track 0.00 -> 36.9 mm, vias 0 -> 2
- net VRTC: track 0.00 -> 35.2 mm, vias 0 -> 2
- net SIM_CLK: track 0.00 -> 34.6 mm
- net 1.8V: track 16.3 -> 46.2 mm, vias 0 -> 4
- net SIM_DATA: track 16.8 -> 43.4 mm
- net GND: track 232.7 -> 241.3 mm

Commit message: completed routing
Routing:
- net UART_TX: track 0.00 -> 98.5 mm, vias 0 -> 4
- net NETSTAT: track 0.00 -> 91.8 mm, vias 0 -> 2
- net POWERSTAT: track 0.00 -> 58.0 mm, vias 0 -> 4
- net SIM_TXD: track 0.00 -> 31.6 mm, vias 0 -> 4
Changed lines of the file:
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@@
     (thickness 1.6)
     (drawings 7)
-    (tracks 621)
+    (tracks 720)
     (zones 0)
     (modules 29)
@@
   (segment (start 73.914 101.854) (end 76.4032 101.854) (width 0.25) (layer F.Cu) (net 29))
   (segment (start 71.501 99.441) (end 73.914 101.854) (width 0.25) (layer F.Cu) (net 29))
+  (segment (start 78.458 78.152) (end 79.14 77.47) (width 0.25) (layer F.Cu) (net 32))
+  (segment (start 77.408 78.152) (end 78.458 78.152) (width 0.25) (layer F.Cu) (net 32))
+  (segment (start 79.14 77.47) (end 81.915 77.47) (width 0.25) (layer F.Cu) (net 32))
+  (via (at 81.915 77.47) (size 0.8) (drill 0.4) (layers F.Cu B.Cu) (net 32))
+  (segment (start 82.314999 77.869999) (end 82.314999 79.737001) (width 0.25) (layer B.Cu) (net 32))
+  (segment (start 81.915 77.47) (end 82.314999 77.869999) (width 0.25) (layer B.Cu) (net 32))
+  (segment (start 82.314999 79.737001) (end 78.232 83.82) (width 0.25) (layer B.Cu) (net 32))
+  (segment (start 78.232 83.82) (end 78.232 86.868) (width 0.25) (layer B.Cu) (net 32))
+  (via (at 78.232 86.868) (size 0.8) (drill 0.4) (layers F.Cu B.Cu) (net 32))
+  (segment (start 78.232 87.433685) (end 77.724 87.941685) (width 0.25) (layer F.Cu) (net 32))
+  (segment (start 78.232 86.868) (end 78.232 87.433685) (width 0.25) (layer F.Cu) (net 32))
+  (segment (start 77.724 87.941685) (end 77.724 93.218) (width 0.25) (layer F.Cu) (net 32))
+  (segment (start 77.724 93.218) (end 75.946 94.996) (width 0.25) (layer F.Cu) (net 32))
+  (via (at 75.946 94.996) (size 0.8) (drill 0.4) (layers F.Cu B.Cu) (net 32))
+  (segment (start 75.546001 95.395999) (end 75.546001 95.776999) (width 0.25) (layer B.Cu) (net 32))
+  (segment (start 75.946 94.996) (end 75.546001 95.395999) (width 0.25) (layer B.Cu) (net 32))
+  (segment (start 75.546001 95.776999) (end 73.787 97.536) (width 0.25) (layer B.Cu) (net 32))
+  (via (at 73.787 97.536) (size 0.8) (drill 0.4) (layers F.Cu B.Cu) (net 32))
+  (segment (start 73.787 97.536) (end 73.787 97.917) (width 0.25) (layer F.Cu) (net 32))
+  (segment (start 73.914 98.044) (end 76.4032 98.044) (width 0.25) (layer F.Cu) (net 32))
+  (segment (start 73.787 97.917) (end 73.914 98.044) (width 0.25) (layer F.Cu) (net 32))
   (segment (start 77.408 79.152) (end 93.503 79.152) (width 0.25) (layer F.Cu) (net 33))
   (segment (start 93.503 79.152) (end 95.631 81.28) (width 0.25) (layer F.Cu) (net 33))
@@
   (segment (start 122.333 70.136) (end 122.333 71.696) (width 0.25) (layer F.Cu) (net 33))
   (segment (start 122.047 69.85) (end 122.333 70.136) (width 0.25) (layer F.Cu) (net 33))
+  (segment (start 83.05941 99.314) (end 83.879401 100.133991) (width 0.25) (layer F.Cu) (net 56))
+  (segment (start 81.5848 99.314) (end 83.05941 99.314) (width 0.25) (layer F.Cu) (net 56))
+  (segment (start 83.879401 100.133991) (end 84.83741 101.092) (width 0.25) (layer F.Cu) (net 56))
+  (segment (start 84.83741 101.092) (end 86.233 101.092) (width 0.25) (layer F.Cu) (net 56))
+  (segment (start 86.233 101.092) (end 87.63 101.092) (width 0.25) (layer F.Cu) (net 56))
+  (segment (start 87.63 101.092) (end 88.265 101.727) (width 0.25) (layer F.Cu) (net 56))
+  (segment (start 88.265 101.727) (end 89.916 101.727) (width 0.25) (layer F.Cu) (net 56))
+  (via (at 89.916 101.727) (size 0.8) (drill 0.4) (layers F.Cu B.Cu) (net 56))
+  (segment (start 89.916 101.727) (end 91.694 101.727) (width 0.25) (layer B.Cu) (net 56))
+  (segment (start 91.694 101.727) (end 93.345 100.076) (width 0.25) (layer B.Cu) (net 56))
+  (segment (start 93.345 100.076) (end 93.345 95.885) (width 0.25) (layer B.Cu) (net 56))
+  (segment (start 93.345 95.885) (end 95.377 93.853) (width 0.25) (layer B.Cu) (net 56))
+  (segment (start 95.377 93.853) (end 98.552 93.853) (width 0.25) (layer B.Cu) (net 56))
+  (segment (start 98.552 93.853) (end 100.076 92.329) (width 0.25) (layer B.Cu) (net 56))
+  (segment (start 100.076 92.329) (end 101.6 92.329) (width 0.25) (layer B.Cu) (net 56))
+  (via (at 101.6 92.329) (size 0.8) (drill 0.4) (layers F.Cu B.Cu) (net 56))
+  (segment (start 101.999999 91.929001) (end 101.999999 88.373001) (width 0.25) (layer F.Cu) (net 56))
+  (segment (start 101.6 92.329) (end 101.999999 91.929001) (width 0.25) (layer F.Cu) (net 56))
+  (segment (start 101.999999 88.373001) (end 102.108 88.265) (width 0.25) (layer F.Cu) (net 56))
+  (via (at 102.108 88.265) (size 0.8) (drill 0.4) (layers F.Cu B.Cu) (net 56))
+  (segment (start 102.108 88.265) (end 102.108 86.614) (width 0.25) (layer B.Cu) (net 56))
+  (segment (start 102.108 86.614) (end 102.108 84.582) (width 0.25) (layer B.Cu) (net 56))
+  (segment (start 102.108 84.582) (end 105.283 81.407) (width 0.25) (layer B.Cu) (net 56))
+  (segment (start 105.283 81.407) (end 105.283 70.358) (width 0.25) (layer B.Cu) (net 56))
+  (segment (start 105.283 70.358) (end 105.537 70.104) (width 0.25) (layer B.Cu) (net 56))
+  (via (at 105.537 70.104) (size 0.8) (drill 0.4) (layers F.Cu B.Cu) (net 56))
+  (segment (start 105.936999 69.704001) (end 105.936999 68.598999) (width 0.25) (layer F.Cu) (net 56))
+  (segment (start 105.537 70.104) (end 105.936999 69.704001) (width 0.25) (layer F.Cu) (net 56))
+  (segment (start 104.49 67.152) (end 101.408 67.152) (width 0.25) (layer F.Cu) (net 56))
+  (segment (start 105.936999 68.598999) (end 104.49 67.152) (width 0.25) (layer F.Cu) (net 56))
+  (segment (start 81.5848 103.124) (end 86.614 103.124) (width 0.25) (layer F.Cu) (net 57))
+  (segment (start 86.614 103.124) (end 87.376 103.886) (width 0.25) (layer F.Cu) (net 57))
+  (segment (start 87.376 103.886) (end 89.027 103.886) (width 0.25) (layer F.Cu) (net 57))
+  (via (at 89.027 103.886) (size 0.8) (drill 0.4) (layers F.Cu B.Cu) (net 57))
+  (segment (start 89.027 103.886) (end 95.885 103.886) (width 0.25) (layer B.Cu) (net 57))
+  (segment (start 95.885 103.886) (end 98.044 101.727) (width 0.25) (layer B.Cu) (net 57))
+  (segment (start 98.044 101.727) (end 114.808 101.727) (width 0.25) (layer B.Cu) (net 57))
+  (segment (start 114.808 101.727) (end 119.761 96.774) (width 0.25) (layer B.Cu) (net 57))
+  (segment (start 119.761 96.774) (end 119.761 94.107) (width 0.25) (layer B.Cu) (net 57))
+  (segment (start 119.761 94.107) (end 117.475 91.821) (width 0.25) (layer B.Cu) (net 57))
+  (segment (start 117.475 91.821) (end 106.172 91.821) (width 0.25) (layer B.Cu) (net 57))
+  (segment (start 106.172 91.821) (end 103.505 89.154) (width 0.25) (layer B.Cu) (net 57))
+  (segment (start 103.505 89.154) (end 103.505 85.344) (width 0.25) (layer B.Cu) (net 57))
+  (segment (start 103.505 85.344) (end 106.553 82.296) (width 0.25) (layer B.Cu) (net 57))
+  (segment (start 106.553 82.296) (end 106.553 82.042) (width 0.25) (layer B.Cu) (net 57))
+  (segment (start 106.553 82.042) (end 106.553 71.374) (width 0.25) (layer B.Cu) (net 57))
+  (segment (start 106.553 71.374) (end 107.442 70.485) (width 0.25) (layer B.Cu) (net 57))
+  (segment (start 107.442 70.485) (end 107.442 68.834) (width 0.25) (layer B.Cu) (net 57))
+  (via (at 107.442 68.834) (size 0.8) (drill 0.4) (layers F.Cu B.Cu) (net 57))
+  (segment (start 107.442 68.268315) (end 106.172 66.998315) (width 0.25) (layer F.Cu) (net 57))
+  (segment (start 107.442 68.834) (end 107.442 68.268315) (width 0.25) (layer F.Cu) (net 57))
+  (segment (start 106.172 66.998315) (end 105.860315 66.998315) (width 0.25) (layer F.Cu) (net 57))
+  (segment (start 105.014 66.152) (end 101.408 66.152) (width 0.25) (layer F.Cu) (net 57))
+  (segment (start 105.860315 66.998315) (end 105.014 66.152) (width 0.25) (layer F.Cu) (net 57))
+  (segment (start 75.3023 99.314) (end 75.0483 99.568) (width 0.25) (layer F.Cu) (net 69))
+  (segment (start 76.4032 99.314) (end 75.3023 99.314) (width 0.25) (layer F.Cu) (net 69))
+  (segment (start 75.0483 99.568) (end 74.041 99.568) (width 0.25) (layer F.Cu) (net 69))
+  (via (at 74.041 99.568) (size 0.8) (drill 0.4) (layers F.Cu B.Cu) (net 69))
+  (segment (start 73.641001 99.967999) (end 73.641001 100.729999) (width 0.25) (layer B.Cu) (net 69))
+  (segment (start 74.041 99.568) (end 73.641001 99.967999) (width 0.25) (layer B.Cu) (net 69))
+  (segment (start 73.641001 100.729999) (end 72.136 102.235) (width 0.25) (layer B.Cu) (net 69))
+  (via (at 72.136 102.235) (size 0.8) (drill 0.4) (layers F.Cu B.Cu) (net 69))
+  (segment (start 71.736001 102.634999) (end 71.736001 105.391001) (width 0.25) (layer F.Cu) (net 69))
+  (segment (start 72.136 102.235) (end 71.736001 102.634999) (width 0.25) (layer F.Cu) (net 69))
+  (segment (start 73.242001 106.897001) (end 122.210999 106.897001) (width 0.25) (layer F.Cu) (net 69))
+  (segment (start 71.736001 105.391001) (end 73.242001 106.897001) (width 0.25) (layer F.Cu) (net 69))
+  (segment (start 122.210999 106.897001) (end 126.111 102.997) (width 0.25) (layer F.Cu) (net 69))
+  (segment (start 126.111 102.997) (end 126.111 99.314) (width 0.25) (layer F.Cu) (net 69))
+  (via (at 126.111 99.06) (size 0.8) (drill 0.4) (layers F.Cu B.Cu) (net 69))
+  (segment (start 126.111 99.314) (end 126.111 99.06) (width 0.25) (layer F.Cu) (net 69))
+  (segment (start 126.111 98.494315) (end 124.333 96.716315) (width 0.25) (layer B.Cu) (net 69))
+  (segment (start 126.111 99.06) (end 126.111 98.494315) (width 0.25) (layer B.Cu) (net 69))
+  (segment (start 124.333 96.716315) (end 124.333 74.549) (width 0.25) (layer B.Cu) (net 69))
+  (via (at 124.333 74.549) (size 0.8) (drill 0.4) (layers F.Cu B.Cu) (net 69))
+  (segment (start 123.933001 74.149001) (end 123.806001 74.149001) (width 0.25) (layer F.Cu) (net 69))
+  (segment (start 124.333 74.549) (end 123.933001 74.149001) (width 0.25) (layer F.Cu) (net 69))
+  (segment (start 123.133 73.476) (end 123.133 71.696) (width 0.25) (layer F.Cu) (net 69))
+  (segment (start 123.806001 74.149001) (end 123.133 73.476) (width 0.25) (layer F.Cu) (net 69))
   (segment (start 117.348 62.23) (end 117.348 60.96) (width 0.25) (layer F.Cu) (net 79))
   (segment (start 117.348 60.96) (end 118.237 60.071) (width 0.25) (layer F.Cu) (net 79))

Commit message: GSM antennae moved to new position
Parts:
- moved J2 8.69 mm to (60.3, 61.1), turned to 180 degrees
Routing:
- net Net-(J2-Pad1): track 77.2 -> 94.3 mm
- net GND: track 241.3 -> 252.8 mm
Changed lines of the file:
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@@
     (thickness 1.6)
     (drawings 7)
-    (tracks 720)
+    (tracks 721)
     (zones 0)
     (modules 29)
@@
   )
   (module custom_footprints:SMA-J-P-H-ST-EM1 (layer F.Cu)
-    (at 68.707 63.373 270)
-    (fp_text reference J2 (at -0.32555 -3.34077 90) (layer F.SilkS)
+    (at 60.325 61.087 180)
+    (fp_text reference J2 (at -0.32555 -3.34077) (layer F.SilkS)
       (effects (font (size 1.001732 1.001732) (thickness 0.015)))
     )
-    (fp_text value SMA-J-P-H-ST-EM1 (at 6.76137 12.36757 90) (layer F.Fab)
+    (fp_text value SMA-J-P-H-ST-EM1 (at 6.76137 12.36757) (layer F.Fab)
       (effects (font (size 1.000205 1.000205) (thickness 0.015)))
     )
@@
     (fp_line (start -3.165 11.42) (end -3.175 1.9) (layer F.Fab) (width 0.127))
     (fp_line (start -5 1.9) (end -3.175 1.9) (layer F.Fab) (width 0.127))
-    (fp_text user PCB~EDGE (at 4.30403 1.70159 90) (layer F.Fab)
+    (fp_text user PCB~EDGE (at 4.30403 1.70159) (layer F.Fab)
       (effects (font (size 0.48045 0.48045) (thickness 0.015)))
     )
@@
     (fp_line (start -3.425 2.15) (end -3.75 2.15) (layer F.CrtYd) (width 0.05))
     (fp_line (start -3.75 2.15) (end -3.75 -2.55) (layer F.CrtYd) (width 0.05))
-    (fp_text user BOARD~THICKNESS:~1.57~MM (at 4.1008 -1.40027 90) (layer F.Fab)
+    (fp_text user BOARD~THICKNESS:~1.57~MM (at 4.1008 -1.40027) (layer F.Fab)
       (effects (font (size 0.480094 0.480094) (thickness 0.015)))
     )
-    (pad 1 smd rect (at 0 0 270) (size 1.27 3.6) (layers F.Cu F.Paste F.Mask)
+    (pad 1 smd rect (at 0 0 180) (size 1.27 3.6) (layers F.Cu F.Paste F.Mask)
       (net 21 "Net-(J2-Pad1)"))
-    (pad 2_1 smd rect (at -2.825 -0.2 270) (size 1.35 4.2) (layers F.Cu F.Paste F.Mask)
-      (net 2 GND))
-    (pad 3_1 smd rect (at 2.825 -0.2 270) (size 1.35 4.2) (layers F.Cu F.Paste F.Mask)
-      (net 2 GND))
-    (pad 2_2 smd rect (at -2.825 -0.2 270) (size 1.35 4.2) (layers B.Cu B.Paste B.Mask)
-      (net 2 GND))
-    (pad 3_2 smd rect (at 2.825 -0.2 270) (size 1.35 4.2) (layers B.Cu B.Paste B.Mask)
+    (pad 2_1 smd rect (at -2.825 -0.2 180) (size 1.35 4.2) (layers F.Cu F.Paste F.Mask)
+      (net 2 GND))
+    (pad 3_1 smd rect (at 2.825 -0.2 180) (size 1.35 4.2) (layers F.Cu F.Paste F.Mask)
+      (net 2 GND))
+    (pad 2_2 smd rect (at -2.825 -0.2 180) (size 1.35 4.2) (layers B.Cu B.Paste B.Mask)
+      (net 2 GND))
+    (pad 3_2 smd rect (at 2.825 -0.2 180) (size 1.35 4.2) (layers B.Cu B.Paste B.Mask)
       (net 2 GND))
   )
@@
   (segment (start 116.967 86.8195) (end 116.3805 86.233) (width 0.25) (layer F.Cu) (net 2))
   (segment (start 116.967 87.63) (end 116.967 86.8195) (width 0.25) (layer F.Cu) (net 2))
-  (segment (start 77.362 66.198) (end 77.408 66.152) (width 0.25) (layer F.Cu) (net 2))
-  (segment (start 68.907 66.198) (end 77.362 66.198) (width 0.25) (layer F.Cu) (net 2))
-  (segment (start 66.557 60.548) (end 66.272 60.833) (width 0.25) (layer F.Cu) (net 2))
-  (segment (start 68.907 60.548) (end 66.557 60.548) (width 0.25) (layer F.Cu) (net 2))
-  (segment (start 66.272 60.833) (end 66.167 60.833) (width 0.25) (layer F.Cu) (net 2))
-  (segment (start 66.167 60.833) (end 64.897 62.103) (width 0.25) (layer F.Cu) (net 2))
-  (segment (start 64.897 62.103) (end 64.897 64.643) (width 0.25) (layer F.Cu) (net 2))
-  (segment (start 66.452 66.198) (end 68.907 66.198) (width 0.25) (layer F.Cu) (net 2))
-  (segment (start 64.897 64.643) (end 66.452 66.198) (width 0.25) (layer F.Cu) (net 2))
   (segment (start 77.408 67.152) (end 77.408 66.152) (width 0.25) (layer F.Cu) (net 2))
   (segment (start 77.408 66.152) (end 77.408 65.152) (width 0.25) (layer F.Cu) (net 2))
@@
   (segment (start 100.33 89.789) (end 99.314 90.805) (width 0.25) (layer F.Cu) (net 2))
   (segment (start 100.33 88.646) (end 100.33 89.789) (width 0.25) (layer F.Cu) (net 2))
+  (segment (start 63.15 65.055) (end 63.15 61.287) (width 0.25) (layer F.Cu) (net 2))
+  (segment (start 64.293 66.198) (end 63.15 65.055) (width 0.25) (layer F.Cu) (net 2))
+  (segment (start 77.408 66.152) (end 77.362 66.198) (width 0.25) (layer F.Cu) (net 2))
+  (segment (start 77.362 66.198) (end 64.293 66.198) (width 0.25) (layer F.Cu) (net 2))
+  (segment (start 64.293 66.198) (end 62.326 66.198) (width 0.25) (layer F.Cu) (net 2))
+  (segment (start 62.326 66.198) (end 60.325 68.199) (width 0.25) (layer F.Cu) (net 2))
+  (segment (start 60.325 68.199) (end 59.436 68.199) (width 0.25) (layer F.Cu) (net 2))
+  (segment (start 57.5 66.263) (end 57.5 61.287) (width 0.25) (layer F.Cu) (net 2))
+  (segment (start 59.436 68.199) (end 57.5 66.263) (width 0.25) (layer F.Cu) (net 2))
   (segment (start 63.33 99.992) (end 63.33 96.454) (width 0.25) (layer F.Cu) (net 3))
   (segment (start 62.103 101.219) (end 63.33 99.992) (width 0.25) (layer F.Cu) (net 3))
@@
   (segment (start 96.266 89.281) (end 97.282 88.265) (width 0.25) (layer B.Cu) (net 16))
   (via (at 97.282 88.265) (size 0.8) (drill 0.4) (layers F.Cu B.Cu) (net 16))
-  (segment (start 70.757 63.373) (end 73.279 60.851) (width 0.25) (layer F.Cu) (net 21))
-  (segment (start 68.707 63.373) (end 70.757 63.373) (width 0.25) (layer F.Cu) (net 21))
-  (segment (start 73.279 60.851) (end 74.15 60.851) (width 0.25) (layer F.Cu) (net 21))
-  (segment (start 74.15 60.851) (end 74.422 60.579) (width 0.25) (layer F.Cu) (net 21))
-  (via (at 74.549 60.452) (size 0.8) (drill 0.4) (layers F.Cu B.Cu) (net 21))
-  (segment (start 74.422 60.579) (end 74.549 60.452) (width 0.25) (layer F.Cu) (net 21))
   (segment (start 74.549 60.452) (end 75.184 59.817) (width 0.25) (layer B.Cu) (net 21))
   (segment (start 75.184 59.817) (end 103.632 59.817) (width 0.25) (layer B.Cu) (net 21))
@@
   (segment (start 103.631 81.152) (end 101.408 81.152) (width 0.25) (layer F.Cu) (net 21))
   (segment (start 104.756001 82.277001) (end 103.631 81.152) (width 0.25) (layer F.Cu) (net 21))
+  (segment (start 74.549 60.452) (end 74.041 60.452) (width 0.25) (layer B.Cu) (net 21))
+  (segment (start 74.041 60.452) (end 66.04 68.453) (width 0.25) (layer B.Cu) (net 21))
+  (segment (start 66.04 68.453) (end 61.849 68.453) (width 0.25) (layer B.Cu) (net 21))
+  (segment (start 61.849 68.453) (end 60.198 66.802) (width 0.25) (layer B.Cu) (net 21))
+  (via (at 60.198 66.802) (size 0.8) (drill 0.4) (layers F.Cu B.Cu) (net 21))
+  (segment (start 60.198 61.214) (end 60.325 61.087) (width 0.25) (layer F.Cu) (net 21))
+  (segment (start 60.198 66.802) (end 60.198 61.214) (width 0.25) (layer F.Cu) (net 21))
   (segment (start 117.348 65.991314) (end 118.999 67.642314) (width 0.25) (layer B.Cu) (net 22))
   (segment (start 117.348 64.77) (end 117.348 65.991314) (width 0.25) (layer B.Cu) (net 22))
