File: SIM808_CIRCUIT.kicad_pcb (KiCad board)
At the start: 2 copper layers, 94 x 49.7 mm, 29 parts, among them J1 USB_B_Micro, J2 SMA-J-P-H-ST-EM1, J3 SIM_Card, J4 AVR-ISP-6, SW1 SW_Push, SW2 SW_Push, U1 MCP73811T-420I-OT, U2 SIM808, U3 74ABT125D, U4 ATmega328-AU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

Commit message: circuit board layout
Parts:
- added H1: MountingHole, MountingHole:MountingHole_3.5mm, F.Cu at (138.8, 63.8)
- added H2: MountingHole, MountingHole:MountingHole_3.5mm, F.Cu at (59.2, 103.9)
- added H3: MountingHole, MountingHole:MountingHole_3.5mm, F.Cu at (136.1, 100.8)
- added H4: MountingHole, MountingHole:MountingHole_3.5mm, F.Cu at (66.8, 62.4)
- added J5: U.FL-R-SMT(01), custom_footprints:HRS_U.FL-R-SMT(01), F.Cu at (54.1, 74.9)
- J1: footprint Connector_USB:USB_Micro-B_GCT_USB3076-30-A -> Connector_USB:USB_Micro-B_Molex-105017-0001
- J2: value SMA-J-P-H-ST-EM1 -> SMA-J-P-H-RA-TH1; footprint custom_footprints:SMA-J-P-H-ST-EM1 -> custom_footprints:SAMTEC_SMA-J-P-H-RA-TH1
- J3: value SIM_Card -> 693012040811; footprint Connector_Card:microSIM_JAE_SF53S006VCBR2000 -> custom_footprints:WURTH_693012040811; moved to B.Cu
- U2: footprint XCVR_SIM808 -> custom_footprints:XCVR_SIM808
- moved J2 5.71 mm to (54.9, 62.7), turned to 0 degrees
- moved J3 4.84 mm to (64.5, 78.4), turned to 180 degrees
- moved J1 1.97 mm to (53.5, 97.4)
Connections:
- U2 pad 35: Net-(J2-Pad1) -> Net-(J5-Pad3)
- U2 pad 66: Net-(U2-Pad66) -> Net-(J2-Pad1)
Routing:
- net Net-(J5-Pad3): track 0.00 -> 104.5 mm, vias 0 -> 2
- net Net-(J2-Pad1): track 94.3 -> 44.0 mm, vias 2 -> 1
- net GND: track 252.8 -> 300.1 mm, vias 0 -> 3
- net SIM_DATA: track 43.4 -> 55.8 mm, vias 2 -> 3
- net SIM_RST: track 43.0 -> 52.5 mm, vias 4 -> 5
- net SIM_CLK: track 34.6 -> 43.9 mm, vias 0 -> 1
- net 1.8V: track 46.2 -> 50.3 mm, vias 4 -> 5
- net RING: track 36.9 -> 40.7 mm, vias 2 -> 4
- net +5V: track 162.1 -> 164.2 mm
- net Net-(J1-Pad4): track 0.00 -> 0.89 mm
