File: SIM808_CIRCUIT.sch (KiCad schematic (older format))
At the start: 29 parts, among them J1 USB_B_Micro, J2 SMA-J-P-H-ST-EM1, J3 SIM_Card, J4 AVR-ISP-6, SW1 SW_Push, SW2 SW_Push, U1 MCP73811T-420I-OT, U2 SIM808, U3 74ABT125D, U4 ATmega328-AU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

Commit message: connected ISP line to AVR
Parts:
- J3: footprint (none) -> Connector_Card:microSIM_JAE_SF53S006VCBR2000
Connections:
- net AVR_RST: now also J4.5 (~RST)
- net MISO: now also J4.1 (MISO)
- net MOSI: now also J4.4 (MOSI)
Changed lines of the file:
@@
 F 0 "J3" H 7580 1300 50  0000 L CNN
 F 1 "SIM_Card" H 7580 1209 50  0000 L CNN
-F 2 "" H 6950 1550 50  0001 C CNN
+F 2 "Connector_Card:microSIM_JAE_SF53S006VCBR2000" H 6950 1550 50  0001 C CNN
 F 3 " ~" H 6900 1200 50  0001 C CNN
 	1    6950 1200
 	1    0    0    -1
 $EndComp
+Wire Wire Line
+	10850 1700 10950 1700
+Wire Wire Line
+	10850 1800 10950 1800
+Text GLabel 10800 2300 2    50   Input ~ 0
+AVR_RST
+Wire Wire Line
+	10800 2300 10800 2100
+Wire Wire Line
+	10800 2100 10850 2100
+Wire Wire Line
+	10850 2100 10850 2000
 $EndSCHEMATC

Commit message: circuit board schematic
Parts:
- removed J2: SMA-J-P-H-ST-EM1, custom_footprints:SMA-J-P-H-ST-EM1, symbol SMA_CONNECTOR:SMA-J-P-H-ST-EM1
- removed J3: SIM_Card, Connector_Card:microSIM_JAE_SF53S006VCBR2000, symbol Connector:SIM_Card
- added H1, H2, H3, H4: MountingHole, MountingHole:MountingHole_3.5mm, symbol Mechanical:MountingHole
- added J2: SMA-J-P-H-RA-TH1, custom_footprints:SAMTEC_SMA-J-P-H-RA-TH1, symbol RIGHT_ANGLE_SMA:SMA-J-P-H-RA-TH1
- added J3: 693012040811, custom_footprints:WURTH_693012040811, symbol NANO_SIM_TRAY:693012040811
- added J5: U.FL-R-SMT(01), custom_footprints:HRS_U.FL-R-SMT(01), symbol UFL_CONNECTOR:U.FL-R-SMT(01)
- J1: footprint Connector_USB:USB_Micro-B_GCT_USB3076-30-A -> Connector_USB:USB_Micro-B_Molex-105017-0001
- U2: footprint XCVR_SIM808 -> custom_footprints:XCVR_SIM808
Connections:
- net 1.8V: now also J3.C1 (1_VCC)
- net GND: now also J2.2 (GND), J2.3 (GND), J2.4 (GND), J2.5 (GND), J3.C5 (5_GND), J5.1 (GND), J5.2 (GND)
- net SIM_CLK: now also J3.C3 (3_CLK)
- net SIM_DATA: now also J3.C7 (7_I/O)
- net SIM_RST: now also J3.C2 (2_RST)
- net at U2.35 (GPS_ANT): now also J5.3 (SIG)
- net at U2.66 (GSM_ANT): now also J2.1 (SIGNAL)
Changed lines of the file:
@@
 EESchema Schematic File Version 4
+LIBS:SIM808_CIRCUIT-cache
 EELAYER 29 0
 EELAYER END
@@
 F 0 "U2" H 3150 5265 50  0000 C CNN
 F 1 "SIM808" H 3150 5174 50  0000 C CNN
-F 2 "XCVR_SIM808" H 3150 3200 50  0001 L BNN
+F 2 "custom_footprints:XCVR_SIM808" H 3150 3200 50  0001 L BNN
 F 3 "" H 3150 3200 50  0001 L BNN
 F 4 "1.03" H 3150 3200 50  0001 L BNN "Field4"
@@
 	1    0    0    -1
 $EndComp
-$Comp
-L SMA_CONNECTOR:SMA-J-P-H-ST-EM1 J2
-U 1 1 5E70A18C
-P 4750 2050
-F 0 "J2" V 4811 2280 50  0000 L CNN
-F 1 "SMA-J-P-H-ST-EM1" V 4902 2280 50  0000 L CNN
-F 2 "custom_footprints:SMA-J-P-H-ST-EM1" H 4750 2050 50  0001 L BNN
-F 3 "" H 4750 2050 50  0001 L BNN
-F 4 "G" H 4750 2050 50  0001 L BNN "Field4"
-F 5 "Samtec" H 4750 2050 50  0001 L BNN "Field5"
-	1    4750 2050
-	0    1    1    0
-$EndComp
 Text GLabel 4550 2450 0    50   Input ~ 0
 GND
 Wire Wire Line
 	4550 2450 4650 2450
-Wire Wire Line
-	4750 2450 4750 2600
-Wire Wire Line
-	4750 2600 3950 2600
 $Comp
 L Connector:USB_B_Micro J1
@@
 F 0 "J1" H 1007 6867 50  0000 C CNN
 F 1 "USB_B_Micro" H 1007 6776 50  0000 C CNN
-F 2 "Connector_USB:USB_Micro-B_GCT_USB3076-30-A" H 1100 6350 50  0001 C CNN
+F 2 "Connector_USB:USB_Micro-B_Molex-105017-0001" H 1100 6350 50  0001 C CNN
 F 3 "~" H 1100 6350 50  0001 C CNN
 	1    950  6400
@@
 Wire Wire Line
 	9400 3850 9250 3850
-Wire Wire Line
-	6250 1400 6450 1400
-Wire Wire Line
-	6000 1200 6450 1200
-Wire Wire Line
-	6250 1100 6450 1100
-Wire Wire Line
-	6250 1000 6450 1000
 $Comp
 L power:GND #PWR0111
@@
 Text GLabel 6250 1000 0    50   Input ~ 0
 SIM_RST
-Wire Wire Line
-	6250 900  6450 900
 Text GLabel 6250 900  0    50   Input ~ 0
 1.8V
 Text GLabel 6250 1400 0    50   Input ~ 0
 SIM_DATA
-$Comp
-L Connector:SIM_Card J3
-U 1 1 5E712AFB
-P 6950 1200
-F 0 "J3" H 7580 1300 50  0000 L CNN
-F 1 "SIM_Card" H 7580 1209 50  0000 L CNN
-F 2 "Connector_Card:microSIM_JAE_SF53S006VCBR2000" H 6950 1550 50  0001 C CNN
-F 3 " ~" H 6900 1200 50  0001 C CNN
-	1    6950 1200
-	1    0    0    -1
-$EndComp
 Wire Wire Line
 	10850 1700 10950 1700
@@
 Wire Wire Line
 	10850 2100 10850 2000
+$Comp
+L RIGHT_ANGLE_SMA:SMA-J-P-H-RA-TH1 J2
+U 1 1 5E811558
+P 4900 1800
+F 0 "J2" V 4961 2030 50  0000 L CNN
+F 1 "SMA-J-P-H-RA-TH1" V 5052 2030 50  0000 L CNN
+F 2 "custom_footprints:SAMTEC_SMA-J-P-H-RA-TH1" H 4900 1800 50  0001 L BNN
+F 3 "" H 4900 1800 50  0001 L BNN
+F 4 "Manufacturer recommendations" H 4900 1800 50  0001 L BNN "Field4"
+F 5 "K" H 4900 1800 50  0001 L BNN "Field5"
+	1    4900 1800
+	0    1    1    0
+$EndComp
+Wire Wire Line
+	4650 2450 4650 2350
+Wire Wire Line
+	4650 2200 4800 2200
+$Comp
+L NANO_SIM_TRAY:693012040811 J3
+U 1 1 5E835CA5
+P 7450 1150
+F 0 "J3" H 7780 1246 50  0000 L CNN
+F 1 "693012040811" H 7780 1155 50  0000 L CNN
+F 2 "custom_footprints:WURTH_693012040811" H 7450 1150 50  0001 L BNN
+F 3 "" H 7450 1150 50  0001 L BNN
+F 4 "Wurth Electronics" H 7450 1150 50  0001 L BNN "Field4"
+F 5 "1.8mm" H 7450 1150 50  0001 L BNN "Field5"
+F 6 "G" H 7450 1150 50  0001 L BNN "Field6"
+	1    7450 1150
+	1    0    0    -1
+$EndComp
+Wire Wire Line
+	6250 900  6750 900
+Wire Wire Line
+	6750 900  6750 850
+Wire Wire Line
+	6750 850  6950 850
+Wire Wire Line
+	6250 1000 6750 1000
+Wire Wire Line
+	6750 1000 6750 950
+Wire Wire Line
+	6750 950  6950 950
+Wire Wire Line
+	6250 1100 6800 1100
+Wire Wire Line
+	6800 1100 6800 1050
+Wire Wire Line
+	6800 1050 6950 1050
+Wire Wire Line
+	6000 1200 6850 1200
+Wire Wire Line
+	6850 1200 6850 1150
+Wire Wire Line
+	6850 1150 6950 1150
+Wire Wire Line
+	6250 1400 6950 1400
+Wire Wire Line
+	6950 1400 6950 1350
+$Comp
+L Mechanical:MountingHole H3
+U 1 1 5E88EBD5
+P 6450 2400
+F 0 "H3" H 6550 2446 50  0000 L CNN
+F 1 "MountingHole" H 6550 2355 50  0000 L CNN
+F 2 "MountingHole:MountingHole_3.5mm" H 6450 2400 50  0001 C CNN
+F 3 "~" H 6450 2400 50  0001 C CNN
+	1    6450 2400
+	1    0    0    -1
+$EndComp
+$Comp
+L Mechanical:MountingHole H1
+U 1 1 5E88F302
+P 6400 2750
+F 0 "H1" H 6500 2796 50  0000 L CNN
+F 1 "MountingHole" H 6500 2705 50  0000 L CNN
+F 2 "MountingHole:MountingHole_3.5mm" H 6400 2750 50  0001 C CNN
+F 3 "~" H 6400 2750 50  0001 C CNN
+	1    6400 2750
+	1    0    0    -1
+$EndComp
+$Comp
+L Mechanical:MountingHole H2
+U 1 1 5E88F52C
+P 6400 3250
+F 0 "H2" H 6500 3296 50  0000 L CNN
+F 1 "MountingHole" H 6500 3205 50  0000 L CNN
+F 2 "MountingHole:MountingHole_3.5mm" H 6400 3250 50  0001 C CNN
+F 3 "~" H 6400 3250 50  0001 C CNN
+	1    6400 3250
+	1    0    0    -1
+$EndComp
+$Comp
+L Mechanical:MountingHole H4
+U 1 1 5E88F7F1
+P 7250 3000
+F 0 "H4" H 7350 3046 50  0000 L CNN
+F 1 "MountingHole" H 7350 2955 50  0000 L CNN
+F 2 "MountingHole:MountingHole_3.5mm" H 7250 3000 50  0001 C CNN
+F 3 "~" H 7250 3000 50  0001 C CNN
+	1    7250 3000
+	1    0    0    -1
+$EndComp
+$Comp
+L power:GND #PWR0123
+U 1 1 5E8931F7
+P 6450 3550
+F 0 "#PWR0123" H 6450 3300 50  0001 C CNN
+F 1 "GND" H 6455 3377 50  0000 C CNN
+F 2 "" H 6450 3550 50  0001 C CNN
+F 3 "" H 6450 3550 50  0001 C CNN
+	1    6450 3550
+	1    0    0    -1
+$EndComp
+Wire Wire Line
+	6450 3550 6450 3250
+Wire Wire Line
+	6450 3250 6400 3250
+$Comp
+L power:GND #PWR0124
+U 1 1 5E89961D
+P 7300 3200
+F 0 "#PWR0124" H 7300 2950 50  0001 C CNN
+F 1 "GND" H 7305 3027 50  0000 C CNN
+F 2 "" H 7300 3200 50  0001 C CNN
+F 3 "" H 7300 3200 50  0001 C CNN
+	1    7300 3200
+	1    0    0    -1
+$EndComp
+$Comp
+L power:GND #PWR0125
+U 1 1 5E899A22
+P 6200 2850
+F 0 "#PWR0125" H 6200 2600 50  0001 C CNN
+F 1 "GND" H 6205 2677 50  0000 C CNN
+F 2 "" H 6200 2850 50  0001 C CNN
+F 3 "" H 6200 2850 50  0001 C CNN
+	1    6200 2850
+	1    0    0    -1
+$EndComp
+$Comp
+L power:GND #PWR0126
+U 1 1 5E899D1B
+P 6200 2400
+F 0 "#PWR0126" H 6200 2150 50  0001 C CNN
+F 1 "GND" H 6205 2227 50  0000 C CNN
+F 2 "" H 6200 2400 50  0001 C CNN
+F 3 "" H 6200 2400 50  0001 C CNN
+	1    6200 2400
+	1    0    0    -1
+$EndComp
+Wire Wire Line
+	6200 2850 6200 2750
+Wire Wire Line
+	6200 2750 6400 2750
+Wire Wire Line
+	6200 2400 6450 2400
+Wire Wire Line
+	7300 3200 7300 3000
+Wire Wire Line
+	7300 3000 7250 3000
+Wire Wire Line
+	3950 2400 4900 2400
+Wire Wire Line
+	4900 2400 4900 2200
+$Comp
+L UFL_CONNECTOR:U.FL-R-SMT(01) J5
+U 1 1 5E8CE870
+P 5550 2250
+F 0 "J5" H 5752 2290 50  0000 L CNN
+F 1 "U.FL-R-SMT(01)" H 5752 2199 50  0000 L CNN
+F 2 "custom_footprints:HRS_U.FL-R-SMT(01)" H 5550 2250 50  0001 L BNN
+F 3 "" H 5550 2250 50  0001 L BNN
+F 4 "Good" H 5550 2250 50  0001 L BNN "Field4"
+F 5 "0.84 USD" H 5550 2250 50  0001 L BNN "Field5"
+F 6 "None" H 5550 2250 50  0001 L BNN "Field6"
+F 7 "U.FL Series 6 Ghz 50 Ohm Ultra-small SMT Coaxial Cable Receptacle" H 5550 2250 50  0001 L BNN "Field7"
+F 8 "U.FL-R-SMT(01)" H 5550 2250 50  0001 L BNN "Field8"
+	1    5550 2250
+	1    0    0    -1
+$EndComp
+Wire Wire Line
+	5150 2150 4950 2150
+Wire Wire Line
+	4950 2150 4950 2600
+Wire Wire Line
+	4950 2600 3950 2600
+Wire Wire Line
+	5150 2350 4650 2350
+Connection ~ 4650 2350
+Wire Wire Line
+	4650 2350 4650 2200
 $EndSCHEMATC
